File: SmartEVCoupler.kicad_pcb (KiCad board)
At the start: 2 copper layers, 100 x 80 mm, 37 parts, among them J1 Type2-Wallbox-IN, J2 Type2-Car-OUT, Q1 IRLZ44NPBF

Commit message: Use deterministic UUIDs for PCB zones; regenerate schematic/pcb
https://claude.ai/code/session_01HtYCFycwjAHofQsQUDsT5P
Parts:
- removed the R_PP at (20.0, 72.0) (x2)
- added R_PP (x2): 2.7kΩ, evc:R_0402, F.Cu at (20.0, 72.0)
